File: Maiskolben_Selfmade/Maiskolben_THT.brd (EAGLE design)
At the start: 72.2 x 80.8 mm, 33 parts, among them IC1 OPA703PA, J2 AUDIO_JACK_5PEBS_35, Q1 IRF5305, Q2 2N7000, U1 CD4050DIP16, U2 ARDUINO_NANOR3

Commit message: Push to HW V1.3
Closes #3, adds drill file (whoops), adds optional LM7805 for v > 12V
Parts:
- added IC2: 7805TV, linear:TO220V
- added R6: 100K, SparkFun-Resistors:AXIAL-0.3
- added SJ1: DIRECT VIN, SparkFun-Passives:PAD-JUMPER-2-NO_YES_SILK
- added U$2: (no value), rgb_matrix:MAISKOLBEN
- added U$4: (no value), creative-commons:BY_TPLACE
- added U$5: (no value), creative-commons:SA_TPLACE
- added U$6: (no value), creative-commons:NC_TPLACE
- added U$7: (no value), creative-commons:CC_TPLACE
- R2, R8: value 5K6 -> 5k6
- R4: value 68K -> 68k
Connections:
- new net A_VIN: SJ1.1, U2.VIN
- net +5V: now also IC2.3
- net DGND: now also IC2.2, R6.P$1
- net OPA+: now also R6.P$2
- net VIN: now also IC2.1, SJ1.2; no longer U2.VIN
Routing:
- net +5V: track 75.8 -> 91.4 mm
- net A_VIN: track 0.00 -> 10.1 mm
- net N$2: track 0.00 -> 7.50 mm
- net OPA+: track 8.76 -> 16.1 mm
Other:
- board text added: "12V max LM7805: 24V max"
- board text added: "Abstützen"
- board text added: "Direct VIN (No LM7805)"
- board text added: "LM7805"
- board text added: "Maiskolben THT 1.3"
- board text removed: "Maiskolben THT 1.1"
Changed lines of the file:
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@@
 <setting verticaltext="up"/>
 </settings>
-<grid distance="12.5" unitdist="mil" unit="mil" style="dots" multiple="1" display="yes" altdistance="0.0125" altunitdist="inch" altunit="inch"/>
+<grid distance="1" unitdist="mm" unit="mm" style="dots" multiple="1" display="yes" altdistance="0.0125" altunitdist="inch" altunit="inch"/>
 <layers>
 <layer number="1" name="Top" color="4" fill="1" visible="yes" active="yes"/>
@@
 <wire x1="61.739" y1="25.5" x2="61.739" y2="29" width="0.4064" layer="21" style="shortdash"/>
 <wire x1="61.1915" y1="60.3175" x2="64.1915" y2="63.3175" width="0.4064" layer="21" style="shortdash"/>
-<text x="18.239" y="78.5" size="1.6764" layer="21" ratio="12">Maiskolben THT 1.1</text>
+<text x="18.239" y="78.5" size="1.6764" layer="21" ratio="12">Maiskolben THT 1.3</text>
 <text x="14.239" y="21" size="1.016" layer="21">Drahtbrücke
 oder bereits durch Taster gebrückt</text>
@@
 <text x="13.239" y="50.5" size="1.016" layer="21" rot="R180">KB 3 SPRS</text>
 <text x="51.239" y="37.5" size="1.016" layer="21" rot="R90" align="center">74HC4050</text>
+<text x="9.8425" y="18.7325" size="1.27" layer="21" ratio="16" rot="R90" align="center-left">Abstützen</text>
+<text x="20.955" y="69.85" size="1.016" layer="22" rot="MR0" align="top-center">Direct VIN
+(No LM7805)</text>
+<text x="3.4925" y="61.595" size="1.016" layer="21" align="top-center">12V max
+LM7805:
+24V max</text>
+<text x="10.16" y="80.01" size="1.016" layer="21" align="top-center">LM7805</text>
 </plain>
 <attributes>
@@
 </element>
 <element name="R7" library="SparkFun-Resistors" package="AXIAL-0.3" value="100R" x="27.9646" y="48.4922" rot="R270"/>
-<element name="R4" library="SparkFun-Resistors" package="AXIAL-0.3" value="68K" x="33.1898" y="40.4105" rot="R270"/>
+<element name="R4" library="SparkFun-Resistors" package="AXIAL-0.3" value="68k" x="33.1898" y="40.4105" rot="R270"/>
 <element name="C7" library="SparkFun-Capacitors" package="CAP-PTH-SMALLEZ" value="100nF" x="27.992" y="30.9345" smashed="yes" rot="R270">
 <attribute name="NAME" x="26.8425" y="31.0805" size="0.8" layer="25" font="vector" ratio="15" rot="R180"/>
 <attribute name="VALUE" x="28.0045" y="32.592" size="0.8" layer="27" font="vector" ratio="15" rot="R90"/>
 </element>
-<element name="R8" library="SparkFun-Resistors" package="AXIAL-0.3" value="5K6" x="19.707" y="48.5074" rot="R270"/>
+<element name="R8" library="SparkFun-Resistors" package="AXIAL-0.3" value="5k6" x="19.707" y="48.5074" rot="R270"/>
 <element name="C8" library="SparkFun-Capacitors" package="CAP-PTH-SMALLEZ" value="10nF" x="25.471" y="44.6914" smashed="yes" rot="R90">
 <attribute name="NAME" x="26.086" y="49.4964" size="0.8" layer="25" font="vector" ratio="15" rot="R180"/>
@@
 </element>
 <element name="R5" library="SparkFun-Resistors" package="AXIAL-0.3" value="1k" x="67.5968" y="48.3104" rot="R270"/>
-<element name="R2" library="SparkFun-Resistors" package="AXIAL-0.3" value="5K6" x="35.3616" y="40.3978" rot="R90"/>
+<element name="R2" library="SparkFun-Resistors" package="AXIAL-0.3" value="5k6" x="35.3616" y="40.3978" rot="R90"/>
 <element name="C6" library="SparkFun-Capacitors" package="CAP-PTH-SMALLEZ" value="10nF" x="38.0936" y="44.1822" smashed="yes" rot="R270">
 <attribute name="NAME" x="37.391" y="45.609" size="0.8" layer="25" font="vector" ratio="15"/>
@@
 </element>
 <element name="U$1" library="rgb_matrix" package="HANNIO_MEDIUM" value="HANNIO_MEDIUM" x="4.739" y="10.5"/>
+<element name="R6" library="SparkFun-Resistors" package="AXIAL-0.3" value="100K" x="31.75" y="51.1175" rot="R270"/>
+<element name="U$2" library="rgb_matrix" package="MAISKOLBEN" value="" x="47.625" y="7.9375"/>
+<element name="IC2" library="linear" package="TO220V" value="7805TV" x="10.16" y="78.74"/>
+<element name="SJ1" library="SparkFun-Passives" package="PAD-JUMPER-2-NO_YES_SILK" value="DIRECT VIN" x="14.9225" y="68.58" rot="MR0"/>
+<element name="U$4" library="creative-commons" package="BY_TPLACE" value="" x="44" y="48" rot="MR0"/>
+<element name="U$5" library="creative-commons" package="SA_TPLACE" value="" x="55" y="48" rot="MR0"/>
+<element name="U$6" library="creative-commons" package="NC_TPLACE" value="" x="66" y="48" rot="MR0"/>
+<element name="U$7" library="creative-commons" package="CC_TPLACE" value="" x="55" y="63" rot="MR0"/>
 </elements>
 <signals>
@@
 <vertex x="-0.125" y="-0.8015"/>
 </polygon>
+<contactref element="R6" pad="P$1"/>
+<contactref element="IC2" pad="2"/>
 </signal>
 <signal name="+5V">
@@
 <wire x1="23.507" y1="54.732" x2="26.829" y2="54.732" width="0.8128" layer="16"/>
 <wire x1="13.739" y1="59" x2="13.739" y2="62.745" width="0.8128" layer="16"/>
-<wire x1="13.739" y1="62.745" x2="27.305" y2="76.2" width="0.8128" layer="16"/>
+<wire x1="13.739" y1="62.745" x2="23.955646875" y2="72.878053125" width="0.8128" layer="16"/>
+<wire x1="23.955646875" y1="72.878053125" x2="27.305" y2="76.2" width="0.8128" layer="16"/>
 <wire x1="27.305" y1="76.2" x2="27.305" y2="76.92" width="0.8128" layer="16"/>
 <wire x1="27.305" y1="76.92" x2="27.279" y2="76.92" width="0.8128" layer="16"/>
@@
 <wire x1="23.507" y1="54.732" x2="23.507" y2="53.268" width="0.6096" layer="16"/>
 <wire x1="23.507" y1="53.268" x2="20.989" y2="50.75" width="0.6096" layer="16"/>
+<contactref element="IC2" pad="3"/>
+<wire x1="12.7" y1="76.2" x2="14.9225" y2="78.4225" width="0.4064" layer="16"/>
+<wire x1="14.9225" y1="78.4225" x2="20.32" y2="78.4225" width="0.4064" layer="16"/>
+<wire x1="20.32" y1="78.4225" x2="20.955" y2="77.7875" width="0.4064" layer="16"/>
+<wire x1="20.955" y1="77.7875" x2="20.955" y2="75.8825" width="0.4064" layer="16"/>
+<wire x1="20.955" y1="75.8825" x2="23.955646875" y2="72.881853125" width="0.4064" layer="16"/>
+<wire x1="23.955646875" y1="72.881853125" x2="23.955646875" y2="72.878053125" width="0.4064" layer="16"/>
 </signal>
 <signal name="OPA+">
@@
 <wire x1="25.471" y1="41.7235" x2="25.4645" y2="41.717" width="0.4064" layer="16"/>
 <wire x1="25.471" y1="44.6974" x2="25.471" y2="44.6914" width="0.4064" layer="16"/>
+<contactref element="R6" pad="P$2"/>
+<wire x1="31.75" y1="47.3075" x2="28.0871" y2="47.3075" width="0.4064" layer="16"/>
+<wire x1="28.0871" y1="47.3075" x2="25.471" y2="44.6914" width="0.4064" layer="16"/>
 </signal>
 <signal name="SENSOR">
@@
 </signal>
 <signal name="VIN">
-<contactref element="U2" pad="VIN"/>
 <contactref element="R10" pad="P$1"/>
 <contactref element="Q1" pad="3"/>
 <contactref element="JP1" pad="PWR"/>
-<wire x1="10.689" y1="68.35" x2="19.659" y2="75.82" width="0.8128" layer="16"/>
-<wire x1="19.659" y1="75.82" x2="19.659" y2="76.92" width="0.8128" layer="16"/>
 <wire x1="5.089" y1="41.39" x2="5.089" y2="41.65" width="1.016" layer="16"/>
 <wire x1="5.089" y1="41.65" x2="2.739" y2="43.5" width="1.016" layer="16"/>
@@
 <wire x1="2.239" y1="40.5" x2="3.129" y2="41.39" width="0.4064" layer="16"/>
 <wire x1="3.129" y1="41.39" x2="5.089" y2="41.39" width="0.4064" layer="16"/>
+<contactref element="IC2" pad="1"/>
+<contactref element="SJ1" pad="2"/>
+<wire x1="10.689" y1="68.35" x2="14.2425" y2="68.35" width="0.4064" layer="16"/>
+<wire x1="14.2425" y1="68.35" x2="14.4725" y2="68.58" width="0.4064" layer="16"/>
+<wire x1="10.689" y1="68.35" x2="7.62" y2="71.419" width="0.4064" layer="16"/>
+<wire x1="7.62" y1="71.419" x2="7.62" y2="76.2" width="0.4064" layer="16"/>
 </signal>
 <signal name="DOWN">
@@
 <contactref element="U2" pad="D10"/>
 <contactref element="U1" pad="IN_E"/>
-<wire x1="47.379" y1="41.21" x2="45.739" y2="42.85" width="0.4064" layer="16"/>
-<wire x1="45.739" y1="42.85" x2="45.739" y2="47" width="0.4064" layer="16"/>
-<wire x1="45.739" y1="47" x2="56.739" y2="58" width="0.4064" layer="16"/>
+<wire x1="47.379" y1="41.21" x2="45.4215" y2="43.1675" width="0.4064" layer="16"/>
+<wire x1="45.4215" y1="43.1675" x2="45.4215" y2="46.6825" width="0.4064" layer="16"/>
+<wire x1="45.4215" y1="46.6825" x2="56.739" y2="58" width="0.4064" layer="16"/>
 <wire x1="56.739" y1="58" x2="56.739" y2="62.5" width="0.4064" layer="16"/>
 <wire x1="56.739" y1="62.5" x2="55.614" y2="63.625" width="0.4064" layer="16"/>
@@
 <wire x1="59.9415" y1="58.8525" x2="59.997421875" y2="59.248421875" width="0.4064" layer="16"/>
 </signal>
+<signal name="P1">
+<via x="8.255" y="28.575" extent="1-16" drill="1.1"/>
+<via x="8.255" y="26.035" extent="1-16" drill="1.1"/>
+<via x="8.255" y="23.495" extent="1-16" drill="1.1"/>
+<via x="8.255" y="20.955" extent="1-16" drill="1.1"/>
+<via x="8.255" y="18.415" extent="1-16" drill="1.1"/>
+<wire x1="8.255" y1="26.035" x2="8.255" y2="28.575" width="0" layer="19" extent="1-1"/>
+<wire x1="8.255" y1="23.495" x2="8.255" y2="26.035" width="0" layer="19" extent="1-1"/>
+<wire x1="8.255" y1="20.955" x2="8.255" y2="23.495" width="0" layer="19" extent="1-1"/>
+<wire x1="8.255" y1="18.415" x2="8.255" y2="20.955" width="0" layer="19" extent="1-1"/>
+</signal>
+<signal name="N$2">
+<wire x1="60.0075" y1="59.3725" x2="60.325" y2="59.3725" width="0.4064" layer="1"/>
+<wire x1="60.325" y1="59.3725" x2="65.405" y2="64.4525" width="0.4064" layer="1"/>
+</signal>
+<signal name="A_VIN">
+<contactref element="U2" pad="VIN"/>
+<contactref element="SJ1" pad="1"/>
+<wire x1="15.3725" y1="68.58" x2="19.659" y2="72.8665" width="0.4064" layer="16"/>
+<wire x1="19.659" y1="72.8665" x2="19.659" y2="76.92" width="0.4064" layer="16"/>
+</signal>
 </signals>
